File: Kicad files/Placa_Teste/Placa_Teste.kicad_pcb (KiCad board)
At the start: 2 copper layers, 50.8 x 50.8 mm, 4 parts

Commit message: Atualizando arquivos kicad e .blender
Routing:
- net (no net): track 0.00 -> 81.7 mm
- added copper zone on B.Cu, net (none)
Changed lines of the file:
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@@
   (general
     (thickness 1.6)
-    (drawings 37)
-    (tracks 17)
+    (drawings 43)
+    (tracks 31)
     (zones 0)
     (modules 4)
@@
     (last_trace_width 0.25)
     (trace_clearance 0.2)
-    (zone_clearance 0.508)
+    (zone_clearance 0.1)
     (zone_45_only no)
     (trace_min 0.2)
@@
       (usegerberadvancedattributes false)
       (creategerberjobfile false)
-      (excludeedgelayer true)
-      (linewidth 0.100000)
+      (excludeedgelayer false)
+      (linewidth 0.050000)
       (plotframeref false)
       (viasonmask false)
@@
       (outputformat 5)
       (mirror false)
-      (drillshape 0)
+      (drillshape 2)
       (scaleselection 1)
       (outputdirectory "svg/"))
@@
     )
   )
-  (gr_line (start 153.27 116) (end 148.27 116) (layer F.SilkS) (width 0.2))
-  (gr_line (start 153.27 114) (end 153.27 116) (layer F.SilkS) (width 0.2))
-  (gr_line (start 148.27 114) (end 153.27 114) (layer F.SilkS) (width 0.2))
-  (gr_line (start 148.27 119) (end 148.27 114) (layer F.SilkS) (width 0.2))
+  (gr_poly (pts (xy 173.70806 90.91422) (xy 174.18558 91.12504) (xy 174.41672 91.42222) (xy 174.50308 91.90228) (xy 174.51578 93.24086) (xy 174.498 93.86824) (xy 174.33036 94.33052) (xy 173.941899 94.718823) (xy 173.580902 94.892178) (xy 173.093698 94.972505) (xy 172.366305 94.93885) (xy 171.61637 94.61246) (xy 171.43222 94.10192) (xy 171.3738 92.7354) (xy 171.36364 92.70492) (xy 171.35602 92.25788) (xy 171.40682 91.8591) (xy 171.52112 91.44508) (xy 171.91609 91.06789) (xy 172.40631 90.88755) (xy 173.25848 90.90914)) (layer B.Cu) (width 0.1))
+  (gr_poly (pts (xy 169.96664 90.86596) (xy 170.44416 91.07678) (xy 170.6753 91.37396) (xy 170.76166 91.85402) (xy 170.77436 93.1926) (xy 170.75658 93.81998) (xy 170.58894 94.28226) (xy 170.200479 94.670563) (xy 169.839482 94.843918) (xy 169.352278 94.924245) (xy 168.624885 94.89059) (xy 167.87495 94.5642) (xy 167.6908 94.05366) (xy 167.63238 92.68714) (xy 167.62222 92.65666) (xy 167.6146 92.20962) (xy 167.6654 91.81084) (xy 167.7797 91.39682) (xy 168.17467 91.01963) (xy 168.66489 90.83929) (xy 169.51706 90.86088)) (layer B.Cu) (width 0.1))
+  (gr_poly (pts (xy 166.09314 90.92438) (xy 166.57066 91.1352) (xy 166.8018 91.43238) (xy 166.88816 91.91244) (xy 166.90086 93.25102) (xy 166.88308 93.8784) (xy 166.71544 94.34068) (xy 166.326979 94.728983) (xy 165.965982 94.902338) (xy 165.478778 94.982665) (xy 164.751385 94.94901) (xy 164.00145 94.62262) (xy 163.8173 94.11208) (xy 163.75888 92.74556) (xy 163.74872 92.71508) (xy 163.7411 92.26804) (xy 163.7919 91.86926) (xy 163.9062 91.45524) (xy 164.30117 91.07805) (xy 164.79139 90.89771) (xy 165.64356 90.9193)) (layer B.Cu) (width 0.1))
+  (gr_poly (pts (xy 173.72076 90.90152) (xy 174.19828 91.11234) (xy 174.42942 91.40952) (xy 174.51578 91.88958) (xy 174.52848 93.22816) (xy 174.5107 93.85554) (xy 174.34306 94.31782) (xy 173.954599 94.706123) (xy 173.593602 94.879478) (xy 173.106398 94.959805) (xy 172.379005 94.92615) (xy 171.62907 94.59976) (xy 171.44492 94.08922) (xy 171.3865 92.7227) (xy 171.37634 92.69222) (xy 171.36872 92.24518) (xy 171.41952 91.8464) (xy 171.53382 91.43238) (xy 171.92879 91.05519) (xy 172.41901 90.87485) (xy 173.27118 90.89644)) (layer B.Mask) (width 0.1))
+  (gr_poly (pts (xy 169.96918 90.86342) (xy 170.4467 91.07424) (xy 170.67784 91.37142) (xy 170.7642 91.85148) (xy 170.7769 93.19006) (xy 170.75912 93.81744) (xy 170.59148 94.27972) (xy 170.203019 94.668023) (xy 169.842022 94.841378) (xy 169.354818 94.921705) (xy 168.627425 94.88805) (xy 167.87749 94.56166) (xy 167.69334 94.05112) (xy 167.63492 92.6846) (xy 167.62476 92.65412) (xy 167.61714 92.20708) (xy 167.66794 91.8083) (xy 167.78224 91.39428) (xy 168.17721 91.01709) (xy 168.66743 90.83675) (xy 169.5196 90.85834)) (layer B.Mask) (width 0.1))
+  (gr_poly (pts (xy 166.10584 90.92438) (xy 166.58336 91.1352) (xy 166.8145 91.43238) (xy 166.90086 91.91244) (xy 166.91356 93.25102) (xy 166.89578 93.8784) (xy 166.72814 94.34068) (xy 166.339679 94.728983) (xy 165.978682 94.902338) (xy 165.491478 94.982665) (xy 164.764085 94.94901) (xy 164.01415 94.62262) (xy 163.83 94.11208) (xy 163.77158 92.74556) (xy 163.76142 92.71508) (xy 163.7538 92.26804) (xy 163.8046 91.86926) (xy 163.9189 91.45524) (xy 164.31387 91.07805) (xy 164.80409 90.89771) (xy 165.65626 90.9193)) (layer B.Mask) (width 0.1))
+  (gr_line (start 150.27 117) (end 150.27 118) (layer F.SilkS) (width 0.4))
+  (gr_line (start 146.27 115) (end 148.27 115) (layer F.SilkS) (width 0.4))
+  (gr_line (start 146.27 117) (end 146.27 115) (layer F.SilkS) (width 0.4))
+  (gr_line (start 152.27 117) (end 146.27 117) (layer F.SilkS) (width 0.4))
   (gr_text D2 (at 172.27 114) (layer F.SilkS)
     (effects (font (size 1 1) (thickness 0.2)))
@@
   (gr_line (start 179.07 127) (end 179.07 76.2) (layer Edge.Cuts) (width 0.05))
   (gr_line (start 128.27 127) (end 153.924 127) (layer Edge.Cuts) (width 0.05))
+  (segment (start 161.27 117) (end 138.27 117) (width 0.25) (layer B.Cu) (net 0))
+  (segment (start 138.27 117) (end 137.27 117) (width 0.25) (layer B.Cu) (net 0))
+  (segment (start 137.27 117) (end 133.27 113) (width 0.25) (layer B.Cu) (net 0))
+  (segment (start 161.27 117) (end 164.27 117) (width 0.25) (layer B.Cu) (net 0))
+  (segment (start 164.27 117) (end 170.27 111) (width 0.25) (layer B.Cu) (net 0))
+  (segment (start 170.27 111) (end 170.27 101) (width 0.25) (layer B.Cu) (net 0))
+  (segment (start 139.27 97) (end 139.27 101) (width 0.25) (layer B.Cu) (net 0))
+  (segment (start 139.27 101) (end 138.27 101) (width 0.25) (layer B.Cu) (net 0))
+  (segment (start 138.27 101) (end 135.27 104) (width 0.25) (layer B.Cu) (net 0))
+  (segment (start 155.27 83) (end 155.27 89) (width 0.25) (layer B.Cu) (net 0))
+  (segment (start 164.060729 98) (end 167.978592 94.082137) (width 1) (layer B.Cu) (net 0))
+  (segment (start 162.27 98) (end 163.060729 98) (width 1) (layer B.Cu) (net 0))
+  (segment (start 163.060729 98) (end 164.060729 98) (width 1) (layer B.Cu) (net 0))
+  (segment (start 164.27 83) (end 172.27 83) (width 1) (layer B.Cu) (net 0))
   (segment (start 147.32 104.14) (end 147.32 107.95) (width 0.25) (layer B.Cu) (net 1))
   (segment (start 147.32 107.95) (end 148.59 109.22) (width 0.25) (layer B.Cu) (net 1))
@@
   (segment (start 158.75 109.22) (end 160.02 107.95) (width 0.25) (layer B.Cu) (net 1))
   (segment (start 160.02 107.95) (end 160.02 104.14) (width 0.25) (layer B.Cu) (net 1))
+  (segment (start 149.32 99.79) (end 149.32 104.14) (width 0.25) (layer B.Cu) (net 2))
   (segment (start 135.104 89.916) (end 139.446 89.916) (width 0.25) (layer B.Cu) (net 2))
-  (segment (start 149.32 99.79) (end 149.32 104.14) (width 0.25) (layer B.Cu) (net 2))
   (segment (start 139.446 89.916) (end 149.32 99.79) (width 0.25) (layer B.Cu) (net 2))
+  (segment (start 134.27 85) (end 133.604 85.666) (width 0.25) (layer B.Cu) (net 3))
+  (segment (start 133.604 85.666) (end 133.604 89.916) (width 0.25) (layer B.Cu) (net 3))
   (segment (start 134.27 81) (end 134.27 85) (width 0.25) (layer B.Cu) (net 3))
-  (segment (start 133.604 85.666) (end 133.604 89.916) (width 0.25) (layer B.Cu) (net 3))
-  (segment (start 134.27 85) (end 133.604 85.666) (width 0.25) (layer B.Cu) (net 3))
+  (segment (start 141.89 81) (end 142.94 81) (width 0.25) (layer B.Cu) (net 4))
+  (segment (start 142.94 81) (end 149.27 87.33) (width 0.25) (layer B.Cu) (net 4))
+  (segment (start 149.27 88) (end 149.27 88.31) (width 0.25) (layer B.Cu) (net 4))
+  (segment (start 149.27 87.33) (end 149.27 88.31) (width 0.25) (layer B.Cu) (net 4))
   (segment (start 149.27 88.31) (end 165.1 104.14) (width 0.25) (layer B.Cu) (net 4))
-  (segment (start 149.27 88) (end 149.27 88.31) (width 0.25) (layer B.Cu) (net 4))
   (segment (start 149.27 87.660998) (end 149.27 88) (width 0.25) (layer B.Cu) (net 4))
-  (segment (start 149.27 87.33) (end 149.27 88.31) (width 0.25) (layer B.Cu) (net 4))
-  (segment (start 142.94 81) (end 149.27 87.33) (width 0.25) (layer B.Cu) (net 4))
-  (segment (start 141.89 81) (end 142.94 81) (width 0.25) (layer B.Cu) (net 4))
+  (zone (net 0) (net_name "") (layer B.Cu) (hatch edge 0.508)
+    (connect_pads (clearance 0.1))
+    (min_thickness 0.254)
+    (fill yes (arc_segments 32) (thermal_gap 0.508) (thermal_bridge_width 0.508))
+    (polygon
+      (pts
+        (xy 163.27 101) (xy 179.27 101) (xy 179.27 128) (xy 128.27 127) (xy 128.27 76)
+        (xy 163.27 76)
+      )
+    )
+  )
 )
